Commit message: add: simulate files  to gazebo and rviz

File: src/bumperbot_description/urdf/bumperbot.urdf.xacro (robot description, xacro)
@@ -1,8 +1,19 @@
 <?xml version="1.0"?>
 <robot xmlns:xacro="http://www.ros.org/wiki/xacro" name="bumperbot">
+    <!-- Include Gazebo Parameters -->
+     <!-- importamos bumperbot_description_gazebo, hacemos un codigo mas manejable y limpio -->
+    <xacro:include filename="$(find bumperbot_description)/urdf/bumperbot_gazebo.xacro" />
     <!-- creamos el link padre de todo donde vamos a ir añadiendo las partes del dron -->
     <link name="base_footprint" />
     <!-- vamos añadiendo links -->
     <link name="base_link">
+        <!-- la inercia añade añade la fricción, resistencia de un objeto a cambiar su movimiento de
+        rotación. -->
+        <inertial>
+            <origin xyz="0 0 0.04" rpy="0.0 0.25 0.3" />
+            <mass value="8.2573504e-01" />
+            <inertia ixx="2.2124416e-02" ixy="-1.2294101e-04" ixz="3.4938785e-04"
+                iyy="2.1193702e-02" iyz="-5.0120904e-05" izz="2.0064271e-02" />
+        </inertial>
         <visual>
             <origin xyz="0.0 0.0 0.0" rpy="0.0 0.0 0.0" />
@@ -11,4 +22,10 @@
             </geometry>
         </visual>
+        <collision>
+            <origin xyz="0 0 0" rpy="0 0 0" />
+            <geometry>
+                <mesh filename="package://bumperbot_description/meshes/base_link.STL" />
+            </geometry>
+        </collision>
     </link>
     <joint name="base_joint" type="fixed">
@@ -19,4 +36,11 @@
     <!-- añadimos nuevo link , la rueda derecha trasera -->
     <link name="wheel_rigth_link">
+        <inertial>
+            <origin xyz="0 -0.014 0" rpy="0 0 0" />
+            <mass value="0.0530086090966721" />
+            <inertia ixx="1.88176298336665E-05" ixy="-4.8444933029987E-10"
+                ixz="1.88163708851143E-08" iyy="3.11510738647764E-05" iyz="-6.93560663069607E-11"
+                izz="1.8801969558182E-05" />
+        </inertial>
         <visual>
             <origin xyz="0.0 0.0 0.0" rpy="1.57 0.0 0.0" />
@@ -25,4 +49,10 @@
             </geometry>
         </visual>
+        <collision>
+            <origin xyz="0 -0.015 0" rpy="1.57 0 0" />
+            <geometry>
+                <sphere radius="0.033" />
+            </geometry>
+        </collision>
     </link>
     <!-- el tipo de joint es continuos porque asi rota sobre el padre -->
@@ -36,4 +66,12 @@
     <!-- añadimos rueda izquierda -->
     <link name="wheel_left_link">
+        <inertial>
+            <origin xyz="0 0.014 0" rpy="0 0 0" />
+            <mass value="0.0530086043217644" />
+            <inertia ixx="1.8792911368909E-05" ixy="3.31256392204584E-10"
+                ixz="-1.14082001662767E-08"
+                iyy="3.11510738759073E-05" iyz="-3.60499245082192E-10"
+                izz="1.88266886146847E-05" />
+        </inertial>
         <visual>
             <origin xyz="0.0 0.0 0.0" rpy="-1.57 0.0 0.0" />
@@ -42,4 +80,10 @@
             </geometry>
         </visual>
+        <collision>
+            <origin xyz="0 0.015 0" rpy="-1.57 0 0" />
+            <geometry>
+                <sphere radius="0.033" />
+            </geometry>
+        </collision>
     </link>
     <joint name="wheel_left_joint" type="continuous">
@@ -51,4 +95,12 @@
     </joint>
     <link name="caster_front_link">
+        <inertial>
+            <origin xyz="3.89968128948481E-07 2.40073004698083E-07 0.00219173397061506" rpy="0 0 0" />
+            <mass value="1.44379265037903E-06" />
+            <inertia ixx="7.23075276010246E-11" ixy="-6.10956883467859E-16"
+                ixz="2.22849693525031E-15"
+                iyy="3.8713793085917E-11" iyz="2.93909858781952E-15"
+                izz="1.00967486676306E-10" />
+        </inertial>
         <visual>
             <origin xyz="0.0 0.0 0.0" rpy="0.0 0.0 0.0" />
@@ -57,4 +109,10 @@
             </geometry>
         </visual>
+        <collision>
+            <origin xyz="0 0 0" rpy="0 0 0" />
+            <geometry>
+                <sphere radius="0.005" />
+            </geometry>
+        </collision>
     </link>
     <joint name="caster_front_joint" type="fixed">
@@ -64,4 +122,12 @@
     </joint>
     <link name="caster_rear_link">
+        <inertial>
+            <origin xyz="3.8996812895542E-07 2.40073004698083E-07 0.00219173397061509" rpy="0 0 0" />
+            <mass value="1.44379265037902E-06" />
+            <inertia ixx="7.23075276010246E-11" ixy="-6.10956872363424E-16"
+                ixz="2.22849693527207E-15"
+                iyy="3.87137930859167E-11" iyz="2.939098587861E-15"
+                izz="1.00967486676306E-10" />
+        </inertial>
         <visual>
             <origin xyz="0.0 0.0 0.0" rpy="0.0 0.0 0.0" />
@@ -70,4 +136,10 @@
             </geometry>
         </visual>
+        <collision>
+            <origin xyz="0 0 0" rpy="0 0 0" />
+            <geometry>
+                <sphere radius="0.005" />
+            </geometry>
+        </collision>
     </link>
     <joint name="caster_rear_joint" type="fixed">
@@ -76,3 +148,17 @@
         <origin xyz="-0.04755 0.0 -0.0275" rpy="0.0 0.0 -0.0275" />
     </joint>
+    <!-- Tarea de la leccion 43.5, añadir lata encima del robot -->
+    <link name="can_link" type="fixed">
+        <visual>
+            <origin xyz="-0.03 0.03 0.078" rpy="1.57 0.0 0.0" />
+            <geometry>
+                <mesh filename="package://bumperbot_description/meshes/can.STL" />
+            </geometry>
+        </visual>
+    </link>
+    <joint name="can_joint" type="fixed">
+        <parent link="base_link" />
+        <child link="can_link" />
+        <origin xyz="0.0 0.0 0.0" rpy="0.0 0.0 0.0" />
+    </joint>
 </robot>

Commit message: section  control configuration with gazebo,

File: src/bumperbot_description/urdf/bumperbot.urdf.xacro (robot description, xacro)
@@ -1,9 +1,9 @@
 <?xml version="1.0"?>
-<robot xmlns:xacro="http://www.ros.org/wiki/xacro" name="bumperbot">
+<robot xmlns:xacro="http://ros.org/wiki/xacro" name="bumperbot">
     <xacro:arg name="is_ignition" default="true"/>
     <!-- Include Gazebo Parameters -->
      <!-- importamos bumperbot_description_gazebo, hacemos un codigo mas manejable y limpio -->
     <xacro:include filename="$(find bumperbot_description)/urdf/bumperbot_gazebo.xacro" />
-    <xacro:include filename="$(find bumperbot description)/>urd/bumperbot_ros2_control_xacro"/>
+    <xacro:include filename="$(find bumperbot_description)/urdf/bumperbot_ros2_control.xacro"/>
     <!-- creamos el link padre de todo donde vamos a ir añadiendo las partes del dron -->
     <link name="base_footprint" />
@@ -27,5 +27,5 @@
             <origin xyz="0 0 0" rpy="0 0 0" />
             <geometry>
-                <mesh filename="package://bumperbot_description/meshes/base_link.STL" />
+                <mesh filename="package://bumperbot_description/meshes/base_link.stl" />
             </geometry>
         </collision>

File: src/bumperbot_description/urdf/bumperbot_gazebo.xacro (robot description, xacro)
@@ -10,5 +10,5 @@
         <fdir1>1 0 0</fdir1>
     </gazebo>
-     <gazebo reference="wheel_left_link">
+    <gazebo reference="wheel_left_link">
         <mu1>1000000000000.0</mu1>
         <mu2>1000000000000.0</mu2>
@@ -19,5 +19,5 @@
         <fdir1>1 0 0</fdir1>
     </gazebo>
-     <gazebo reference="caster_front_link">
+    <gazebo reference="caster_front_link">
         <mu1>0.1</mu1>
         <mu2>0.1</mu2>
@@ -26,5 +26,5 @@
         <minDepth>0.001</minDepth>
     </gazebo>
-     <gazebo reference="caster_rear_link">
+    <gazebo reference="caster_rear_link">
         <mu1>0.1</mu1>
         <mu2>0.1</mu2>
@@ -36,15 +36,14 @@
         <!-- añadimos los plugin de ros2 control
         este plugin es por si estamos usando ros2 humble -->
-        <xacro:if value="$(args is_ignition">
-        <plugin filename="ign_ros2_control-system" name="ign_ros2_control::IgnitionROS2ControlPlugin">
-            <parameters>
-            </parameters>
-        </plugin>
+        <xacro:if value="$(arg is_ignition)">
+            <plugin filename="ign_ros2_control-system" name="ign_ros2_control::IgnitionROS2ControlPlugin">
+                <parameters>$(find bumperbot_controller)/config/bumperbot_controllers.yaml</parameters>
+            </plugin>
         </xacro:if>
         <!-- este plugin es por si es jazzy -->
         <xacro:unless value="$(arg is_ignition)">
-            <plugin filename="gz_ros_control-system" name="gz_ros2_control::GazeboSimROS2ControlPlugin">
-                <parameters>
-                </parameters>
+            <plugin filename="gz_ros_control-system"
+                name="gz_ros2_control::GazeboSimROS2ControlPlugin">
+                <parameters>$(find bumperbot_controller)/config/bumperbot_controllers.yaml</parameters>
             </plugin>
         </xacro:unless>

File: src/bumperbot_description/urdf/bumperbot_ros2_control.xacro (robot description, xacro)
@@ -1,13 +1,13 @@
 <?xml version="1.0"?>
-<robot name="bumperbot" xmlns:xacro="htpp://ros.org/wiki/xacro">
+<robot name="bumperbot" xmlns:xacro="http://ros.org/wiki/xacro">
     <!-- Definimos el controller , que va a ser el control total del robot -->
     <ros2_control name="RobotSystem" type="system">
         <!-- Añadimos aqui los plugins que necesita si es humble , jazzy... -->
-        <xacro:if value="$(args is_ignition">
+        <xacro:if value="$(arg is_ignition)">
             <hardware>
                 <plugin>ign_ro2_control/ignition</plugin>
             </hardware>
         </xacro:if>
-        <xacro:unless value="$(args is_ignition)">
+        <xacro:unless value="$(arg is_ignition)">
             <hardware>
                 <plugin>gz_ros2_control/GazeboSimSystem</plugin>
