Commit message: fixed code controller terminal and gazebo terminal working finally

File: src/bumperbot_description/urdf/bumperbot.urdf.xacro (robot description, xacro)
@@ -1,166 +1,145 @@
 <?xml version="1.0"?>
-<robot xmlns:xacro="http://ros.org/wiki/xacro" name="bumperbot">
-    <xacro:arg name="is_ignition" default="true"/>
-    <!-- Include Gazebo Parameters -->
-     <!-- importamos bumperbot_description_gazebo, hacemos un codigo mas manejable y limpio -->
-    <xacro:include filename="$(find bumperbot_description)/urdf/bumperbot_gazebo.xacro" />
-    <xacro:include filename="$(find bumperbot_description)/urdf/bumperbot_ros2_control.xacro"/>
-    <!-- creamos el link padre de todo donde vamos a ir añadiendo las partes del dron -->
-    <link name="base_footprint" />
-    <!-- vamos añadiendo links -->
-    <link name="base_link">
-        <!-- la inercia añade añade la fricción, resistencia de un objeto a cambiar su movimiento de
-        rotación. -->
-        <inertial>
-            <origin xyz="0 0 0.04" rpy="0.0 0.25 0.3" />
-            <mass value="8.2573504e-01" />
-            <inertia ixx="2.2124416e-02" ixy="-1.2294101e-04" ixz="3.4938785e-04"
-                iyy="2.1193702e-02" iyz="-5.0120904e-05" izz="2.0064271e-02" />
-        </inertial>
-        <visual>
-            <origin xyz="0.0 0.0 0.0" rpy="0.0 0.0 0.0" />
-            <geometry>
-                <mesh filename="package://bumperbot_description/meshes/base_link.stl" />
-            </geometry>
-        </visual>
-        <collision>
-            <origin xyz="0 0 0" rpy="0 0 0" />
-            <geometry>
-                <mesh filename="package://bumperbot_description/meshes/base_link.stl" />
-            </geometry>
-        </collision>
-    </link>
-    <joint name="base_joint" type="fixed">
-        <parent link="base_footprint" />
-        <child link="base_link" />
-        <origin xyz="0.0 0.0 0.033" rpy="0.0 0.0 0.033" />
-    </joint>
-    <!-- añadimos nuevo link , la rueda derecha trasera -->
-    <link name="wheel_rigth_link">
-        <inertial>
-            <origin xyz="0 -0.014 0" rpy="0 0 0" />
-            <mass value="0.0530086090966721" />
-            <inertia ixx="1.88176298336665E-05" ixy="-4.8444933029987E-10"
-                ixz="1.88163708851143E-08" iyy="3.11510738647764E-05" iyz="-6.93560663069607E-11"
-                izz="1.8801969558182E-05" />
-        </inertial>
-        <visual>
-            <origin xyz="0.0 0.0 0.0" rpy="1.57 0.0 0.0" />
-            <geometry>
-                <mesh filename="package://bumperbot_description/meshes/wheel_right_link.stl" />
-            </geometry>
-        </visual>
-        <collision>
-            <origin xyz="0 -0.015 0" rpy="1.57 0 0" />
-            <geometry>
-                <sphere radius="0.033" />
-            </geometry>
-        </collision>
-    </link>
-    <!-- el tipo de joint es continuos porque asi rota sobre el padre -->
-    <joint name="wheel_rigth_joint" type="continuous">
-        <parent link="base_link" />
-        <child link="wheel_rigth_link" />
-        <origin xyz="0.0 -0.07 0.0" rpy="0.0 0.0 0.0" />
-        <!-- marcamos el eje de rotacion -->
-        <axis xyz="0.0 1.0 0.0" />
-    </joint>
-    <!-- añadimos rueda izquierda -->
-    <link name="wheel_left_link">
-        <inertial>
-            <origin xyz="0 0.014 0" rpy="0 0 0" />
-            <mass value="0.0530086043217644" />
-            <inertia ixx="1.8792911368909E-05" ixy="3.31256392204584E-10"
-                ixz="-1.14082001662767E-08"
-                iyy="3.11510738759073E-05" iyz="-3.60499245082192E-10"
-                izz="1.88266886146847E-05" />
-        </inertial>
-        <visual>
-            <origin xyz="0.0 0.0 0.0" rpy="-1.57 0.0 0.0" />
-            <geometry>
-                <mesh filename="package://bumperbot_description/meshes/wheel_left_link.stl" />
-            </geometry>
-        </visual>
-        <collision>
-            <origin xyz="0 0.015 0" rpy="-1.57 0 0" />
-            <geometry>
-                <sphere radius="0.033" />
-            </geometry>
-        </collision>
-    </link>
-    <joint name="wheel_left_joint" type="continuous">
-        <parent link="base_link" />
-        <child link="wheel_left_link" />
-        <!-- medida en mm -->
-        <origin xyz="0.0 0.07 0.0" rpy="0.0 0.0 0.0" />
-        <axis xyz="0.0 1.0 0.0" />
-    </joint>
-    <link name="caster_front_link">
-        <inertial>
-            <origin xyz="3.89968128948481E-07 2.40073004698083E-07 0.00219173397061506" rpy="0 0 0" />
-            <mass value="1.44379265037903E-06" />
-            <inertia ixx="7.23075276010246E-11" ixy="-6.10956883467859E-16"
-                ixz="2.22849693525031E-15"
-                iyy="3.8713793085917E-11" iyz="2.93909858781952E-15"
-                izz="1.00967486676306E-10" />
-        </inertial>
-        <visual>
-            <origin xyz="0.0 0.0 0.0" rpy="0.0 0.0 0.0" />
-            <geometry>
-                <mesh filename="package://bumperbot_description/meshes/caster_front_link.stl" />
-            </geometry>
-        </visual>
-        <collision>
-            <origin xyz="0 0 0" rpy="0 0 0" />
-            <geometry>
-                <sphere radius="0.005" />
-            </geometry>
-        </collision>
-    </link>
-    <joint name="caster_front_joint" type="fixed">
-        <parent link="base_link" />
-        <child link="caster_front_link" />
-        <origin xyz="0.04755 0.0 -0.0275" rpy="0.0 0.0 -0.0275" />
-    </joint>
-    <link name="caster_rear_link">
-        <inertial>
-            <origin xyz="3.8996812895542E-07 2.40073004698083E-07 0.00219173397061509" rpy="0 0 0" />
-            <mass value="1.44379265037902E-06" />
-            <inertia ixx="7.23075276010246E-11" ixy="-6.10956872363424E-16"
-                ixz="2.22849693527207E-15"
-                iyy="3.87137930859167E-11" iyz="2.939098587861E-15"
-                izz="1.00967486676306E-10" />
-        </inertial>
-        <visual>
-            <origin xyz="0.0 0.0 0.0" rpy="0.0 0.0 0.0" />
-            <geometry>
-                <mesh filename="package://bumperbot_description/meshes/caster_rear_link.stl" />
-            </geometry>
-        </visual>
-        <collision>
-            <origin xyz="0 0 0" rpy="0 0 0" />
-            <geometry>
-                <sphere radius="0.005" />
-            </geometry>
-        </collision>
-    </link>
-    <joint name="caster_rear_joint" type="fixed">
-        <parent link="base_link" />
-        <child link="caster_rear_link" />
-        <origin xyz="-0.04755 0.0 -0.0275" rpy="0.0 0.0 -0.0275" />
-    </joint>
-    <!-- Tarea de la leccion 43.5, añadir lata encima del robot -->
-    <link name="can_link" type="fixed">
-        <visual>
-            <origin xyz="-0.03 0.03 0.078" rpy="1.57 0.0 0.0" />
-            <geometry>
-                <mesh filename="package://bumperbot_description/meshes/can.STL" />
-            </geometry>
-        </visual>
-    </link>
-    <joint name="can_joint" type="fixed">
-        <parent link="base_link" />
-        <child link="can_link" />
-        <origin xyz="0.0 0.0 0.0" rpy="0.0 0.0 0.0" />
-    </joint>
+<robot name="bumperbot" xmlns:xacro="http://ros.org/wiki/xacro">
+  <!-- Start GZ or Ignition depending on ROS 2 Version -->
+  <xacro:arg name="is_ignition" default="true"/>
+  <!-- Include Gazebo Parameters -->
+  <xacro:include filename="$(find bumperbot_description)/urdf/bumperbot_gazebo.xacro" />
+  <!-- Include ros2_control Plugins -->
+  <xacro:include filename="$(find bumperbot_description)/urdf/bumperbot_ros2_control.xacro" />
+  <link name="base_footprint"/>
+  <link name="base_link">
+    <inertial>
+      <origin xyz="0 0 0.04" rpy="0.0 0.25 0.3" />
+      <mass value="8.2573504e-01"/>
+      <inertia ixx="2.2124416e-02" ixy="-1.2294101e-04" ixz="3.4938785e-04"
+               iyy="2.1193702e-02" iyz="-5.0120904e-05"
+               izz="2.0064271e-02" />
+    </inertial>
+    <visual>
+      <origin xyz="0 0 0" rpy="0 0 0" />
+      <geometry>
+        <mesh filename="package://bumperbot_description/meshes/base_link.STL" />
+      </geometry>
+    </visual>
+    <collision>
+      <origin xyz="0 0 0" rpy="0 0 0" />
+      <geometry>
+        <mesh filename="package://bumperbot_description/meshes/base_link.STL" />
+      </geometry>
+    </collision>
+  </link>
+  <joint name="base_joint" type="fixed">
+    <parent link="base_footprint"/>
+    <child link="base_link" />
+    <origin xyz="0 0 0.033" rpy="0 0 0"/>
+  </joint>
+  <link name="wheel_right_link">
+    <inertial>
+      <origin xyz="0 -0.014 0" rpy="0 0 0" />
+      <mass value="0.0530086090966721" />
+      <inertia ixx="1.88176298336665E-05" ixy="-4.8444933029987E-10" ixz="1.88163708851143E-08"
+               iyy="3.11510738647764E-05" iyz="-6.93560663069607E-11"
+               izz="1.8801969558182E-05" />
+    </inertial>
+    <visual>
+      <origin xyz="0 0 0" rpy="1.57 0 0" />
+      <geometry>
+        <mesh filename="package://bumperbot_description/meshes/wheel_right_link.STL" />
+      </geometry>
+    </visual>
+    <collision>
+      <origin xyz="0 -0.015 0" rpy="1.57 0 0" />
+      <geometry>
+        <sphere radius="0.033"/>
+      </geometry>
+    </collision>
+  </link>
+  <joint name="wheel_right_joint" type="continuous">
+    <origin xyz="0 -0.0701101849418637 0" rpy="0 0 0" />
+    <parent link="base_link" />
+    <child link="wheel_right_link" />
+    <axis xyz="0 1 0" />
+  </joint>
+  <link
+    name="wheel_left_link">
+    <inertial>
+      <origin xyz="0 0.014 0" rpy="0 0 0" />
+      <mass value="0.0530086043217644" />
+      <inertia ixx="1.8792911368909E-05"  ixy="3.31256392204584E-10" ixz="-1.14082001662767E-08"
+               iyy="3.11510738759073E-05" iyz="-3.60499245082192E-10"
+               izz="1.88266886146847E-05" />
+    </inertial>
+    <visual>
+      <origin xyz="0 0 0" rpy="-1.57 0 0" />
+      <geometry>
+        <mesh filename="package://bumperbot_description/meshes/wheel_left_link.STL" />
+      </geometry>
+    </visual>
+    <collision>
+      <origin xyz="0 0.015 0" rpy="-1.57 0 0" />
+      <geometry>
+        <sphere radius="0.033"/>
+      </geometry>
+    </collision>
+  </link>
+  <joint name="wheel_left_joint" type="continuous">
+    <origin xyz="0 0.0701101849418642 0" rpy="0 0 0" />
+    <parent link="base_link" />
+    <child link="wheel_left_link" />
+    <axis xyz="0 1 0" />
+  </joint>
+  <link name="caster_front_link">
+    <inertial>
+      <origin xyz="3.89968128948481E-07 2.40073004698083E-07 0.00219173397061506" rpy="0 0 0" />
+      <mass value="1.44379265037903E-06" />
+      <inertia ixx="7.23075276010246E-11" ixy="-6.10956883467859E-16" ixz="2.22849693525031E-15"
+               iyy="3.8713793085917E-11"  iyz="2.93909858781952E-15"
+               izz="1.00967486676306E-10" />
+    </inertial>
+    <visual>
+      <origin xyz="0 0 0" rpy="0 0 0" />
+      <geometry>
+        <mesh filename="package://bumperbot_description/meshes/caster_front_link.STL" />
+      </geometry>
+    </visual>
+    <collision>
+      <origin xyz="0 0 0" rpy="0 0 0" />
+      <geometry>
+        <sphere radius="0.005"/>
+      </geometry>
+    </collision>
+  </link>
+  <joint name="caster_front_joint" type="fixed">
+    <origin xyz="0.04755 0 -0.0275" rpy="0 0 0" />
+    <parent link="base_link" />
+    <child link="caster_front_link" />
+    <axis xyz="0 0 0" />
+  </joint>
+  <link name="caster_rear_link">
+    <inertial>
+      <origin xyz="3.8996812895542E-07 2.40073004698083E-07 0.00219173397061509" rpy="0 0 0" />
+      <mass value="1.44379265037902E-06" />
+      <inertia ixx="7.23075276010246E-11" ixy="-6.10956872363424E-16" ixz="2.22849693527207E-15"
+               iyy="3.87137930859167E-11" iyz="2.939098587861E-15"
+               izz="1.00967486676306E-10" />
+    </inertial>
+    <visual>
+      <origin xyz="0 0 0" rpy="0 0 0" />
+      <geometry>
+        <mesh filename="package://bumperbot_description/meshes/caster_rear_link.STL" />
+      </geometry>
+    </visual>
+    <collision>
+      <origin xyz="0 0 0" rpy="0 0 0" />
+      <geometry>
+        <sphere radius="0.005"/>
+      </geometry>
+    </collision>
+  </link>
+  <joint name="caster_rear_joint" type="fixed">
+    <origin xyz="-0.04755 0 -0.0275" rpy="0 0 0" />
+    <parent link="base_link" />
+    <child link="caster_rear_link" />
+    <axis xyz="0 0 0" />
+  </joint>
 </robot>

File: src/bumperbot_description/urdf/bumperbot_gazebo.xacro (robot description, xacro)
@@ -1,51 +1,54 @@
 <?xml version="1.0"?>
-<robot name="bumperbot" xmlns:xacro="htpp://www.ros.org/wiki/xacro">
-    <gazebo reference="wheel_right_link">
-        <mu1>1000000000000.0</mu1>
-        <mu2>1000000000000.0</mu2>
-        <kp>100000000000.0</kp>
-        <kd>10.0</kd>
-        <minDepth>0.001</minDepth>
-        <maxVel>0.1</maxVel>
-        <fdir1>1 0 0</fdir1>
-    </gazebo>
-    <gazebo reference="wheel_left_link">
-        <mu1>1000000000000.0</mu1>
-        <mu2>1000000000000.0</mu2>
-        <kp>100000000000.0</kp>
-        <kd>10.0</kd>
-        <minDepth>0.001</minDepth>
-        <maxVel>0.1</maxVel>
-        <fdir1>1 0 0</fdir1>
-    </gazebo>
-    <gazebo reference="caster_front_link">
-        <mu1>0.1</mu1>
-        <mu2>0.1</mu2>
-        <kp>1000000.0</kp>
-        <kd>10.0</kd>
-        <minDepth>0.001</minDepth>
-    </gazebo>
-    <gazebo reference="caster_rear_link">
-        <mu1>0.1</mu1>
-        <mu2>0.1</mu2>
-        <kp>1000000.0</kp>
-        <kd>100.0</kd>
-        <minDepth>0.001</minDepth>
-    </gazebo>
-    <gazebo>
-        <!-- añadimos los plugin de ros2 control
-        este plugin es por si estamos usando ros2 humble -->
-        <xacro:if value="$(arg is_ignition)">
-            <plugin filename="ign_ros2_control-system" name="ign_ros2_control::IgnitionROS2ControlPlugin">
-                <parameters>$(find bumperbot_controller)/config/bumperbot_controllers.yaml</parameters>
-            </plugin>
-        </xacro:if>
-        <!-- este plugin es por si es jazzy -->
-        <xacro:unless value="$(arg is_ignition)">
-            <plugin filename="gz_ros_control-system"
-                name="gz_ros2_control::GazeboSimROS2ControlPlugin">
-                <parameters>$(find bumperbot_controller)/config/bumperbot_controllers.yaml</parameters>
-            </plugin>
-        </xacro:unless>
-    </gazebo>
+<robot name="bumperbot" xmlns:xacro="http://ros.org/wiki/xacro">
+  <!-- Wheels -->
+  <gazebo reference="wheel_left_link">
+    <mu1>1000000000000000.0</mu1>
+    <mu2>1000000000000000.0</mu2>
+    <kp>1000000000000.0</kp>
+    <kd>10.0</kd>
+    <minDepth>0.001</minDepth>
+    <maxVel>0.1</maxVel>
+    <fdir1>1 0 0</fdir1>
+  </gazebo>
+  <gazebo reference="wheel_right_link">
+    <mu1>1000000000000000.0</mu1>
+    <mu2>1000000000000000.0</mu2>
+    <kp>1000000000000.0</kp>
+    <kd>10.0</kd>
+    <minDepth>0.001</minDepth>
+    <maxVel>0.1</maxVel>
+    <fdir1>1 0 0</fdir1>
+  </gazebo>
+  <!-- Caster Wheels -->
+  <gazebo reference="caster_rear_link">
+    <mu1>0.1</mu1>
+    <mu2>0.1</mu2>
+    <kp>1000000.0</kp>
+    <kd>100.0</kd>
+    <minDepth>0.001</minDepth>
+    <maxVel>1.0</maxVel>
+  </gazebo>
+  <gazebo reference="caster_front_link">
+    <mu1>0.1</mu1>
+    <mu2>0.1</mu2>
+    <kp>1000000.0</kp>
+    <kd>100.0</kd>
+    <minDepth>0.001</minDepth>
+    <maxVel>1.0</maxVel>
+  </gazebo>
+  <!-- ROS 2 Control -->
+  <gazebo>
+    <!-- ROS 2 Humble -->
+    <xacro:if value="$(arg is_ignition)">
+      <plugin filename="ign_ros2_control-system" name="ign_ros2_control::IgnitionROS2ControlPlugin">
+        <parameters>$(find bumperbot_controller)/config/bumperbot_controllers.yaml</parameters>
+      </plugin>
+    </xacro:if>
+    <!-- ROS 2 Iron or above -->
+    <xacro:unless value="$(arg is_ignition)">
+      <plugin filename="gz_ros2_control-system" name="gz_ros2_control::GazeboSimROS2ControlPlugin">
+        <parameters>$(find bumperbot_controller)/config/bumperbot_controllers.yaml</parameters>
+      </plugin>
+    </xacro:unless>
+  </gazebo>
 </robot>

File: src/bumperbot_description/urdf/bumperbot_ros2_control.xacro (robot description, xacro)
@@ -1,12 +1,13 @@
 <?xml version="1.0"?>
-<robot name="bumperbot" xmlns:xacro="http://ros.org/wiki/xacro">
-    <!-- Definimos el controller , que va a ser el control total del robot -->
+<robot xmlns:xacro="http://www.ros.org/wiki/xacro" name="bumperbot">
     <ros2_control name="RobotSystem" type="system">
-        <!-- Añadimos aqui los plugins que necesita si es humble , jazzy... -->
+        <!-- ros2_control Gazebo -->
+        <!-- ROS 2 Humble -->
         <xacro:if value="$(arg is_ignition)">
             <hardware>
-                <plugin>ign_ro2_control/ignition</plugin>
+                <plugin>ign_ros2_control/IgnitionSystem</plugin>
             </hardware>
         </xacro:if>
+        <!-- ROS 2 Iron or above -->
         <xacro:unless value="$(arg is_ignition)">
             <hardware>
@@ -14,21 +15,20 @@
             </hardware>
         </xacro:unless>
+        <!-- ros2_control Common Interfaces -->
         <joint name="wheel_right_joint">
-            <!-- aqui podemos darle un valor maximo a la velocidad de las ruedas -->
             <command_interface name="velocity">
-                <param name="min">-1</param>
-                <param name="max">1</param>
+              <param name="min">-1</param>
+              <param name="max">1</param>
             </command_interface>
             <state_interface name="position" />
-            <state_interface name="velocityt" />
+            <state_interface name="velocity" />
         </joint>
         <joint name="wheel_left_joint">
-            <!-- aqui podemos darle un valor maximo a la velocidad de las ruedas -->
             <command_interface name="velocity">
-                <param name="min">-1</param>
-                <param name="max">1</param>
+              <param name="min">-1</param>
+              <param name="max">1</param>
             </command_interface>
             <state_interface name="position" />
-            <state_interface name="velocityt" />
+            <state_interface name="velocity" />
         </joint>
     </ros2_control>

Commit message: create a gazebo bridge and senson imu

File: src/bumperbot_description/urdf/bumperbot.urdf.xacro (robot description, xacro)
@@ -143,3 +143,34 @@
     <axis xyz="0 0 0" />
   </joint>
+  <link name="imu_link">
+    <inertial>
+       <origin xyz="-0.00552433659106688 0.000168210391520346 0.000514000497342681" rpy="0 0 0" />
+       <mass value="0.000528415362211671" />
+       <inertia
+              ixx="1.46176048428261e-08"
+              ixy="1.40015117949421e-10"
+              ixz="-1.99633872937403e-12"
+              iyy="8.59662482954888e-09"
+              iyz="7.52375112767959e-12"
+              izz="2.30279421279312e-08"/>
+    </inertial>
+    <visual>
+      <origin xyz="0.0 0.0 0.0" rpy="0.0 0.0 0.0"/>
+      <geometry>
+        <mesh filename="package://bumperbot_description/meshes/imu_link.STL"/>
+      </geometry>
+    </visual>
+    <collision>
+       <origin xyz="0.0 0.0 0.0" rpy="0.0 0.0 0.0"/>
+      <geometry>
+        <mesh filename="package://bumperbot_description/meshes/imu_link.STL"/>
+      </geometry>
+    </collision>
+  </link>
+  <joint name="imu_joint" type="fixed">
+    <origin xyz="0.0 0.0 0.07" rpy="0.0 0.0 0.0"/>
+   <parent link="base_link"/>
+   <child link="imu_link"/>
+   <axis xyz="0.0 0.0 0.0"/>
+  </joint>
 </robot>

File: src/bumperbot_description/urdf/bumperbot_gazebo.xacro (robot description, xacro)
@@ -44,4 +44,6 @@
         <parameters>$(find bumperbot_controller)/config/bumperbot_controllers.yaml</parameters>
       </plugin>
+      <plugin filename="ignition-gazebo-imu-system" name="ignition::gazebo::systems::Imu">
+      </plugin>
     </xacro:if>
     <!-- ROS 2 Iron or above -->
@@ -50,5 +52,52 @@
         <parameters>$(find bumperbot_controller)/config/bumperbot_controllers.yaml</parameters>
       </plugin>
+      <plugin filename="gz-sim-imu-system" name="gz::sim::systems::Imu"></plugin>
     </xacro:unless>
   </gazebo>
+  <gazebo reference="imu_link">
+    <sensor name="imu" type="imu">
+      <alwaya_rate>true</alwaya_rate>
+      <update_rate>100</update_rate>
+      <gz_frame_id>imu_link</gz_frame_id>
+      <topic>imu</topic>
+      <imu>
+        <angular_velocity >
+          <x>
+            <noise type="gaussian">
+              <mean>0.0</mean>
+              <stddev>2e-4</stddev>
+            </noise>
+          </x>
+          <y>
+             <noise type="gaussian">
+              <mean>0.0</mean>
+              <stddev>2e-4</stddev>
+            </noise>
+          </y>
+          <z>
+             <noise type="gaussian">
+              <mean>0.0</mean>
+              <stddev>2e-4</stddev>
+            </noise>
+          </z>
+        </angular_velocity>
+        <linear_aceleration>
+          <x>
+            <noise type="gaussian">
+              <mean>0.0</mean>
+              <stadev>1.7e-2</stadev>
+            </noise>
+          </x>
+          <y><noise type="gaussian">
+              <mean>0.0</mean>
+              <stadev>1.7e-2</stadev>
+            </noise></y>
+          <z><noise type="gaussian">
+              <mean>0.0</mean>
+              <stadev>1.7e-2</stadev>
+            </noise></z>
+        </linear_aceleration>
+      </imu>
+    </sensor>
+  </gazebo>
 </robot>
